File: PCBs/Controller/Controller/Controller.kicad_pcb (KiCad board)
At the start: 2 copper layers, 48 parts, among them J1 Conn_01x06_Male, J2 BATT_01x02_Male, SW1 SW_Push_Dual, SW2 SW_Push_Dual, SW3 SW_SPDT, SW4 SW_SPDT, U1 LF50_TO220, U2 LF33_TO220, U24L1 NRF24L01_Breakout, U24L2 NRF24L01_Breakout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

Commit message: Finsihed PCB Layout - exported Gerbers v1
Parts:
- moved D4 82.6 mm to (144.8, 69.8)
- moved C2 80.1 mm to (165.1, 53.3), turned to 180 degrees
- moved D2 74.7 mm to (144.8, 77.5)
- moved SW2 71.1 mm to (151.1, 83.2), turned to 90 degrees
- moved U2 69.9 mm to (186.7, 59.7)
- moved R4 69.3 mm to (147.3, 64.8), turned to 90 degrees
- moved R8 69.1 mm to (142.9, 122.6), turned to 180 degrees
- moved C3 68.5 mm to (157.5, 72.4), turned to 90 degrees
- moved U1 68.0 mm to (153.7, 59.7)
- moved U24L2 67.3 mm to (129.5, 77.5), turned to 90 degrees
- moved C1 65.8 mm to (165.1, 67.3), turned to 180 degrees
- moved R1 65.5 mm to (176.5, 83.8), turned to 90 degrees
- moved Y1 62.3 mm to (150.5, 110.5), turned to 270 degrees
- moved U24L1 61.6 mm to (204.5, 77.5), turned to 90 degrees
- moved R2 58.8 mm to (151.1, 72.4), turned to 90 degrees
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Connections:
- net /CTS renamed Net-(J1-Pad2)
- net /DTR renamed DTR
- D5 pad 2: RX -> TX
- J1 pad 3: 5V -> VCC
- J1 pad 5: RX -> TX
- U6 pad H2: A3 -> A5
- U6 pad V2: A2 -> A4
- U7 pad 27: A2 -> A4
- U7 pad 28: A3 -> A5
- U7 pad 3: RX -> TX
Routing:
- net D4: track 0.00 -> 180.6 mm
- net D13: track 0.00 -> 160.3 mm, vias 0 -> 2
- net D8: track 0.00 -> 150.3 mm
- net D11: track 0.00 -> 134.4 mm
- net D7: track 0.00 -> 127.9 mm
- net D12: track 0.00 -> 117.5 mm
- net 5V: track 0.00 -> 110.6 mm, vias 0 -> 5
- net 3V3: track 0.00 -> 108.1 mm
- net TX: track 0.00 -> 98.7 mm
- net D5: track 0.00 -> 93.7 mm, vias 0 -> 2
- net RX: track 0.00 -> 84.7 mm
- net D3: track 0.00 -> 68.1 mm, vias 0 -> 2
- net A5: track 0.00 -> 67.3 mm, vias 0 -> 2
- net DTR: track 0.00 -> 60.5 mm
- net A0: track 0.00 -> 60.3 mm, vias 0 -> 2
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- added copper zone on F.Cu, net 5V
- added copper zone on B.Cu, net GND
Other:
- board outline added: 91.4 x 77.5 mm
- rule trace_min: 0.2 -> 0.25
