File: PCBs/Controller/Controller/Controller.sch (KiCad schematic (older format))
At the start: 48 parts, among them J1 Conn_01x06_Male, J2 BATT_01x02_Male, SW1 SW_Push_Dual, SW2 SW_Push_Dual, SW3 SW_SPDT, SW4 SW_SPDT, U1 LF50_TO220, U2 LF33_TO220, U24L1 NRF24L01_Breakout, U24L2 NRF24L01_Breakout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

Commit message: Properly replaced Joystick schematic
all footprints should be good
Solution was found at path
https://github.com/benwis/SparkFun-Kicad-Libraries/blob/master/SparkFun-Electromechanical.pretty/JOYSTICK.kicad_mod
Parts:
- U5, U6: footprint Controller:JOYSTICK -> Joystick:JOYSTICK
Changed lines of the file:
@@
 F 0 "U5" H 8000 1780 59  0000 L BNN
 F 1 "JOYSTICKLEFT" H 8000 550 59  0000 L BNN
-F 2 "Controller:JOYSTICK" H 8300 1250 50  0001 C CNN
+F 2 "Joystick:JOYSTICK" H 8300 1250 50  0001 C CNN
 F 3 "" H 8300 1250 50  0001 C CNN
 	1    8300 1250
@@
 F 0 "U6" H 9550 1830 59  0000 L BNN
 F 1 "JOYSTICKRIGHT" H 9550 600 59  0000 L BNN
-F 2 "Controller:JOYSTICK" H 9850 1300 50  0001 C CNN
+F 2 "Joystick:JOYSTICK" H 9850 1300 50  0001 C CNN
 F 3 "" H 9850 1300 50  0001 C CNN
 	1    9850 1300

Commit message: Footprints and netlist generated without errors - ready for pcb development
Parts:
- SW1, SW2: symbol Switch:SW_Push_Dual -> Buttons:SW_Push_Dual
Changed lines of the file:
@@
 $EndComp
 $Comp
-L Switch:SW_Push_Dual SW2
+L Buttons:SW_Push_Dual SW2
 U 1 1 5C5121E4
 P 4250 3450
@@
 $EndComp
 $Comp
-L Switch:SW_Push_Dual SW1
+L Buttons:SW_Push_Dual SW1
 U 1 1 5C512256
 P 4150 4150
@@
 Text GLabel 1900 6350 2    50   Input ~ 0
 D10
+Wire Wire Line
+	4050 3650 4050 3450
+Wire Wire Line
+	4450 3650 4450 3450
+Connection ~ 4450 3450
+Wire Wire Line
+	4350 4350 4350 4150
+Connection ~ 4350 4150
+Wire Wire Line
+	3950 4350 3950 4150
 $EndSCHEMATC

Commit message: Finsihed PCB Layout - exported Gerbers v1
Connections:
- net 5V: no longer J1.3 (Pin_3)
- net A2: no longer U6.V2 (V), U7.27 (A4)
- net A3: no longer U6.H2 (H), U7.28 (A5)
- net RX: no longer D5.2 (A), J1.5 (Pin_5), U7.3 (D1_TX)
- net CTS: no longer names the net of J1.2 (Pin_2)
- new net A4: U6.V2 (V), U7.27 (A4)
- new net A5: U6.H2 (H), U7.28 (A5)
- new net TX: D5.2 (A), J1.5 (Pin_5), U7.3 (D1_TX)
- new net VCC: J1.3 (Pin_3)
Changed lines of the file:
@@
 Wire Wire Line
 	7600 1250 7600 850
-Text Label 7300 850  0    70   ~ 0
-VCC
 Connection ~ 7600 850
 Wire Wire Line
@@
 	7500 1250 7300 1250
 Connection ~ 7500 1250
-Text Label 7300 1250 0    70   ~ 0
-GND
 Wire Wire Line
 	7900 950  7800 950
-Text Label 7800 950  0    70   ~ 0
-V1
 Wire Wire Line
 	7900 1350 7800 1350
-Text Label 7800 1350 0    70   ~ 0
-H1
 $Comp
 L Controller-eagle-import:JOYSTICKPTH U5
@@
 Wire Wire Line
 	9150 1300 9150 900
-Text Label 8850 900  0    70   ~ 0
-VCC
 Connection ~ 9150 900
 Wire Wire Line
@@
 	9050 1300 8850 1300
 Connection ~ 9050 1300
-Text Label 8850 1300 0    70   ~ 0
-GND
 Wire Wire Line
 	9450 1000 9350 1000
-Text Label 9350 1000 0    70   ~ 0
-V1
 Wire Wire Line
 	9450 1400 9350 1400
-Text Label 9350 1400 0    70   ~ 0
-H1
 $Comp
 L Controller-eagle-import:JOYSTICKPTH U6
@@
 	1    0    0    -1
 $EndComp
-Text Label 5200 2100 0    50   ~ 0
-DTR
-Text Label 5200 2000 0    50   ~ 0
-RX
-Text Label 5200 1800 0    50   ~ 0
-VCC
-Text Label 5200 1900 0    50   ~ 0
-TX
-Text Label 5200 1700 0    50   ~ 0
-CTS
-Text Label 5200 1600 0    50   ~ 0
-GND
 Text GLabel 5450 1600 2    50   Input ~ 0
 GND
@@
 Wire Wire Line
 	3950 4350 3950 4150
+Text GLabel 5450 2100 2    50   Input ~ 0
+DTR
 $EndSCHEMATC

Commit message: Reduced complexity, removed 1 rf module
Parts:
- removed U24L2: NRF24L01_Breakout, RF_Module:nRF24L01_Breakout, symbol RF:NRF24L01_Breakout
- SW1, SW2: symbol Buttons:SW_Push_Dual -> Controller-rescue:SW_Push_Dual-Buttons
- U3: symbol Potentiometers:PTA4543 -> Controller-rescue:PTA4543-Potentiometers
- U4: symbol Potentiometers:P090S -> Controller-rescue:P090S-Potentiometers
- U7: symbol ATMega:ATmega328P-PU-DIP28 -> Controller-rescue:ATmega328P-PU-DIP28-ATMega
Connections:
- net RF2: no longer SW4.1 (A)
Changed lines of the file:
@@
-$EndComp
-$Comp
-L RF:NRF24L01_Breakout U24L2
-U 1 1 5C511EB3
-P 10750 4350
-F 0 "U24L2" H 11228 4328 50  0000 L CNN
-F 1 "NRF24L01_Breakout" H 11228 4237 50  0000 L CNN
-F 2 "RF_Module:nRF24L01_Breakout" H 10900 4950 50  0001 L CIN
-F 3 "http://www.nordicsemi.com/eng/content/download/2730/34105/file/nRF24L01_Product_Specification_v2_0.pdf" H 10750 4250 50  0001 C CNN
-	1    10750 4350
-	1    0    0    -1
 $EndComp
 $Comp
@@
 $EndComp
 $Comp
-L Buttons:SW_Push_Dual SW2
+L Controller-rescue:SW_Push_Dual-Buttons SW2
 U 1 1 5C5121E4
 P 4250 3450
@@
 $EndComp
 $Comp
-L Buttons:SW_Push_Dual SW1
+L Controller-rescue:SW_Push_Dual-Buttons SW1
 U 1 1 5C512256
 P 4150 4150
@@
 $EndComp
 $Comp
-L Potentiometers:P090S U4
+L Controller-rescue:P090S-Potentiometers U4
 U 1 1 5C51439A
 P 7650 3000
@@
 $EndComp
 $Comp
-L Potentiometers:PTA4543 U3
+L Controller-rescue:PTA4543-Potentiometers U3
 U 1 1 5C51450A
 P 7550 3900
@@
 $EndComp
 $Comp
-L ATMega:ATmega328P-PU-DIP28 U7
+L Controller-rescue:ATmega328P-PU-DIP28-ATMega U7
 U 1 1 5C525263
 P 6150 3300
@@
 Text GLabel 10200 2900 1    50   Input ~ 0
 3V3
-Text GLabel 10750 4950 3    50   Input ~ 0
-GND
 Wire Wire Line
 	5650 300  6200 300
@@
 Text GLabel 7500 2850 0    50   Input ~ 0
 A1
-Text GLabel 10250 4650 0    50   Input ~ 0
-D8
-Text GLabel 10250 4550 0    50   Input ~ 0
-D7
-Text GLabel 10250 4250 0    50   Input ~ 0
-D13
-Text GLabel 10250 4150 0    50   Input ~ 0
-D12
-Text GLabel 10250 4050 0    50   Input ~ 0
-D11
 Text GLabel 7800 950  0    50   Input ~ 0
 A2
@@
 Wire Wire Line
 	9300 3300 10100 3300
-Wire Wire Line
-	10300 3300 10300 3750
-Wire Wire Line
-	10300 3750 10750 3750
 $Comp
 L Connector:Conn_01x06_Male J1
@@
 Text GLabel 9300 3650 0    50   Input ~ 0
 RF1
-Text GLabel 10300 3550 0    50   Input ~ 0
-RF2
 Text GLabel 1900 3300 2    50   Input ~ 0
 RF1
