File: PCBs/Receiver/Receiver/Receiver.kicad_pcb (KiCad board)
At the start: 2 copper layers, 96.5 x 96.5 mm, 51 parts, among them J1 ESC_CTL_1, J10 Servo_2, J11 Conn_01x06_Male, J12 HCS04_Header, J13 Raw_Batt_Header, J14 GEN_Header, J15 Accel_1, J2 ESC_CTL_2, J3 ESC_CTL_3, J4 ESC_CTL_4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

Commit message: Rev 1.1 of Receiver Board - added mounts and cutouts for seperation
Parts:
- added G***: LOGO, Logo:WE_logo_5mm, F.Cu at (174.6, 58.4)
- moved J14 24.9 mm to (156.7, 100.3)
- moved J5 7.87 mm to (103.9, 38.1), turned to 0 degrees
- moved J8 7.62 mm to (190.5, 124.5), turned to 180 degrees
- moved J11 4.85 mm to (115.3, 71.6)
- moved R10 2.54 mm to (119.4, 80.0)
- moved R5 2.54 mm to (129.5, 83.8)
- moved C3 2.34 mm to (119.1, 69.3)
Routing:
- net VDD: track 16.5 -> 60.4 mm
- net D10: track 31.3 -> 11.1 mm
- net GND: track 30.0 -> 47.0 mm, vias 1 -> 3
- net 5V: track 23.0 -> 29.6 mm
- net RX: track 37.1 -> 31.0 mm
- net TX: track 35.8 -> 30.3 mm
- net Net-(D5-Pad1): track 6.81 -> 4.27 mm
- net RST: track 43.6 -> 41.5 mm
- net 3V3: track 97.5 -> 95.4 mm
- net Net-(D10-Pad1): track 57.2 -> 57.3 mm, vias 1 -> 2
- net (no net): vias 0 -> 3
Other:
- outline, holes or cut-outs redrawn
- net class HP: clearance 0.8 -> 0.4
- board text added: "4DX2 Receiver Rev 1.1"
- board text added: "Board made by Will Ehman"

Commit message: Aesthetic Updates to prep for manu
Parts:
- added G***: LOGO, Logo:Big HexB, F.Cu at (149.9, 81.3)
